Commit message: Increased effort limits for the wheels

File: vetex_support/urdf/vetex_macro.xacro (robot description, xacro)
@@ -127,5 +127,5 @@
       <child link="${prefix}left_front_wheel" />
       <axis xyz="0 1 0" />
-      <limit effort="0" velocity="3" />
+      <limit effort="20" velocity="3" />
     </joint>
     <joint name="${prefix}left_rear_wheel_joint" type="continuous">
@@ -135,5 +135,5 @@
       <child link="${prefix}left_rear_wheel" />
       <axis xyz="0 1 0" />
-      <limit effort="0" velocity="3" />
+      <limit effort="20" velocity="3" />
     </joint>
     <joint name="${prefix}right_rear_wheel_joint" type="continuous">
@@ -143,5 +143,5 @@
       <child link="${prefix}right_rear_wheel" />
       <axis xyz="0 1 0" />
-      <limit effort="0" velocity="3" />
+      <limit effort="20" velocity="3" />
     </joint>
     <joint name="${prefix}right_front_wheel_joint" type="continuous">
@@ -151,5 +151,5 @@
       <child link="${prefix}right_front_wheel" />
       <axis xyz="0 1 0" />
-      <limit effort="0" velocity="3" />
+      <limit effort="20" velocity="3" />
     </joint>
     <!-- end of joint list -->
