Commit message: Added changes for colors

File: euler_support/urdf/euler_macro.xacro (robot description, xacro)
@@ -30,7 +30,7 @@
 		</collision>
 		<inertial>
-      <mass value="0.1"/>
+      <mass value="1.0"/>
       <origin xyz="0 0 0"/>
-      <inertia ixx="1.0" ixy="0.0" ixz="0.0" iyy="1.0" iyz="0.0" izz="1.0"/>
+      <inertia ixx="0.01" ixy="0.0" ixz="0.0" iyy="0.01" iyz="0.0" izz="0.01"/>
     </inertial>
 	</link>
@@ -52,7 +52,7 @@
 		</collision>
 		<inertial>
-      <mass value="0.1"/>
+      <mass value="1.0"/>
       <origin xyz="0 0 0"/>
-      <inertia ixx="1.0" ixy="0.0" ixz="0.0" iyy="1.0" iyz="0.0" izz="1.0"/>
+      <inertia ixx="0.01" ixy="0.0" ixz="0.0" iyy="0.01" iyz="0.0" izz="0.01"/>
     </inertial>
 	</link>
@@ -74,7 +74,7 @@
 		</collision>
 		<inertial>
-      <mass value="0.1"/>
+      <mass value="1.0"/>
       <origin xyz="0 0 0"/>
-      <inertia ixx="1.0" ixy="0.0" ixz="0.0" iyy="1.0" iyz="0.0" izz="1.0"/>
+      <inertia ixx="0.01" ixy="0.0" ixz="0.0" iyy="0.01" iyz="0.0" izz="0.01"/>
     </inertial>
 	</link>
@@ -94,7 +94,7 @@
 		</collision>
 		<inertial>
-      <mass value="0.1"/>
+      <mass value="0.3"/>
       <origin xyz="0 0 0"/>
-      <inertia ixx="1.0" ixy="0.0" ixz="0.0" iyy="1.0" iyz="0.0" izz="1.0"/>
+      <inertia ixx="0.001" ixy="0.0" ixz="0.0" iyy="0.001" iyz="0.0" izz="0.001"/>
     </inertial>
 	</link>
@@ -116,5 +116,5 @@
       <mass value="0.1"/>
       <origin xyz="0 0 0"/>
-      <inertia ixx="1.0" ixy="0.0" ixz="0.0" iyy="1.0" iyz="0.0" izz="1.0"/>
+      <inertia ixx="0.001" ixy="0.0" ixz="0.0" iyy="0.001" iyz="0.0" izz="0.001"/>
     </inertial>
 	</link>
@@ -136,5 +136,5 @@
       <mass value="0.1"/>
       <origin xyz="0 0 0"/>
-      <inertia ixx="1.0" ixy="0.0" ixz="0.0" iyy="1.0" iyz="0.0" izz="1.0"/>
+      <inertia ixx="0.001" ixy="0.0" ixz="0.0" iyy="0.001" iyz="0.0" izz="0.001"/>
     </inertial>
 	</link>

File: motoman_mh5lf_support/urdf/mh5lf_macro.xacro (robot description, xacro)
@@ -24,7 +24,7 @@
 			</collision>
 			<inertial>
-		      <mass value="0.1"/>
+		      <mass value="1.0"/>
 		      <origin xyz="0 0 0"/>
-		      <inertia ixx="1.0" ixy="0.0" ixz="0.0" iyy="1.0" iyz="0.0" izz="1.0"/>
+		      <inertia ixx="0.05" ixy="0.0" ixz="0.0" iyy="0.05" iyz="0.0" izz="0.05"/>
 		    </inertial>
 		</link>
@@ -45,7 +45,7 @@
 			</collision>
 			<inertial>
-		      <mass value="0.1"/>
+		      <mass value="1.0"/>
 		      <origin xyz="0 0 0"/>
-		      <inertia ixx="1.0" ixy="0.0" ixz="0.0" iyy="1.0" iyz="0.0" izz="1.0"/>
+		      <inertia ixx="0.05" ixy="0.0" ixz="0.0" iyy="0.05" iyz="0.0" izz="0.05"/>
 		    </inertial>
 		</link>
@@ -64,7 +64,7 @@
 			</collision>
 			<inertial>
-		      <mass value="0.1"/>
+		      <mass value="1.0"/>
 		      <origin xyz="0 0 0"/>
-		      <inertia ixx="1.0" ixy="0.0" ixz="0.0" iyy="1.0" iyz="0.0" izz="1.0"/>
+		      <inertia ixx="0.05" ixy="0.0" ixz="0.0" iyy="0.05" iyz="0.0" izz="0.05"/>
 		    </inertial>
 		</link>
@@ -83,7 +83,7 @@
 			</collision>
 			<inertial>
-		      <mass value="0.1"/>
+		      <mass value="1.0"/>
 		      <origin xyz="0 0 0"/>
-		      <inertia ixx="1.0" ixy="0.0" ixz="0.0" iyy="1.0" iyz="0.0" izz="1.0"/>
+		      <inertia ixx="0.05" ixy="0.0" ixz="0.0" iyy="0.05" iyz="0.0" izz="0.05"/>
 		    </inertial>
 		</link>
@@ -102,7 +102,7 @@
 			</collision>
 			<inertial>
-		      <mass value="0.1"/>
+		      <mass value="1.0"/>
 		      <origin xyz="0 0 0"/>
-		      <inertia ixx="1.0" ixy="0.0" ixz="0.0" iyy="1.0" iyz="0.0" izz="1.0"/>
+		      <inertia ixx="0.05" ixy="0.0" ixz="0.0" iyy="0.05" iyz="0.0" izz="0.05"/>
 		    </inertial>
 		</link>
@@ -121,7 +121,7 @@
 			</collision>
 			<inertial>
-		      <mass value="0.1"/>
+		      <mass value="1.0"/>
 		      <origin xyz="0 0 0"/>
-		      <inertia ixx="1.0" ixy="0.0" ixz="0.0" iyy="1.0" iyz="0.0" izz="1.0"/>
+		      <inertia ixx="0.05" ixy="0.0" ixz="0.0" iyy="0.05" iyz="0.0" izz="0.05"/>
 		    </inertial>
 		</link>
@@ -140,7 +140,7 @@
 			</collision>
 			<inertial>
-		      <mass value="0.1"/>
+		      <mass value="1.0"/>
 		      <origin xyz="0 0 0"/>
-		      <inertia ixx="1.0" ixy="0.0" ixz="0.0" iyy="1.0" iyz="0.0" izz="1.0"/>
+		      <inertia ixx="0.05" ixy="0.0" ixz="0.0" iyy="0.05" iyz="0.0" izz="0.05"/>
 		    </inertial>
 		</link>

File: vetex_support/urdf/vetex_macro.xacro (robot description, xacro)
@@ -14,9 +14,9 @@
       <collision>
         <geometry>
-          <mesh filename="package://vetex_support/meshes/collision/base_link.stl" />
+          <mesh filename="package://vetex_support/meshes/visual/base_link.stl" />
         </geometry>
       </collision>
       <inertial>
-        <mass value="0.1"/>
+        <mass value="52.0"/>
         <origin xyz="0 0 0"/>
         <inertia ixx="1.0" ixy="0.0" ixz="0.0" iyy="1.0" iyz="0.0" izz="1.0"/>
@@ -35,4 +35,5 @@
       </visual>
       <collision>
+        <origin xyz="0 0 0" rpy="1.5708 0 0" />
         <geometry>
           <cylinder length="0.2" radius="0.2"/>
@@ -41,7 +42,7 @@
       </collision>
       <inertial>
-        <mass value="0.1"/>
+        <mass value="5.8517"/>
         <origin xyz="0 0 0"/>
-        <inertia ixx="1.0" ixy="0.0" ixz="0.0" iyy="1.0" iyz="0.0" izz="1.0"/>
+        <inertia ixx="0.0501" ixy="0.0" ixz="0.0" iyy="0.0501" iyz="0.0" izz="0.0501"/>
       </inertial>
     </link>
@@ -55,4 +56,5 @@
       </visual>
       <collision>
+        <origin xyz="0 0 0" rpy="1.5708 0 0" />
         <geometry>
           <cylinder length="0.2" radius="0.2"/>
@@ -61,7 +63,7 @@
       </collision>
       <inertial>
-        <mass value="0.1"/>
+        <mass value="5.8517"/>
         <origin xyz="0 0 0"/>
-        <inertia ixx="1.0" ixy="0.0" ixz="0.0" iyy="1.0" iyz="0.0" izz="1.0"/>
+        <inertia ixx="0.0501" ixy="0.0" ixz="0.0" iyy="0.0501" iyz="0.0" izz="0.0501"/>
       </inertial>
     </link>
@@ -76,5 +78,6 @@
         </visual>
       <collision>
-        <origin rpy="3.1415 0 0" />
+        <origin xyz="0 0 0" rpy="1.5708 0 0" />
+        <!--<origin rpy="3.1415 0 0" />-->
         <geometry>
           <cylinder length="0.2" radius="0.2"/>
@@ -83,7 +86,7 @@
       </collision>
       <inertial>
-        <mass value="0.1"/>
+        <mass value="5.8517"/>
         <origin xyz="0 0 0"/>
-        <inertia ixx="1.0" ixy="0.0" ixz="0.0" iyy="1.0" iyz="0.0" izz="1.0"/>
+        <inertia ixx="0.0501" ixy="0.0" ixz="0.0" iyy="0.0501" iyz="0.0" izz="0.0501"/>
       </inertial>
     </link>
@@ -98,5 +101,6 @@
       </visual>
       <collision>
-        <origin rpy="3.1415 0 0" />
+        <origin xyz="0 0 0" rpy="1.5708 0 0" />
+        <!--<origin rpy="3.1415 0 0" />-->
         <geometry>
           <cylinder length="0.2" radius="0.2"/>
@@ -105,7 +109,7 @@
       </collision>
       <inertial>
-        <mass value="0.1"/>
+        <mass value="5.8517"/>
         <origin xyz="0 0 0"/>
-        <inertia ixx="1.0" ixy="0.0" ixz="0.0" iyy="1.0" iyz="0.0" izz="1.0"/>
+        <inertia ixx="0.0501" ixy="0.0" ixz="0.0" iyy="0.0501" iyz="0.0" izz="0.0501"/>
       </inertial>
     </link>
@@ -118,5 +122,6 @@
     </joint>
     <joint name="${prefix}left_front_wheel_joint" type="continuous">
-      <origin xyz="0 0.58668 0.21577" rpy="1.57 1 0" />
+      <!--<origin xyz="0 0.58668 0.21577" rpy="1.57 1 0" />-->
+      <origin xyz="0 0.58668 0.21577" rpy="0 0 0" />
       <parent link="${prefix}base_link" />
       <child link="${prefix}left_front_wheel" />
@@ -125,5 +130,6 @@
     </joint>
     <joint name="${prefix}left_rear_wheel_joint" type="continuous">
-      <origin xyz="-2.0878 0.58642 0.21577" rpy="1.57 1 0" />
+      <!--<origin xyz="-2.0878 0.58642 0.21577" rpy="1.57 1 0" />-->
+      <origin xyz="-2.0878 0.58642 0.21577" rpy="0 0 0" />
       <parent link="${prefix}base_link" />
       <child link="${prefix}left_rear_wheel" />
@@ -132,5 +138,6 @@
     </joint>
     <joint name="${prefix}right_rear_wheel_joint" type="continuous">
-      <origin xyz="-2.0878 -0.58668 0.21577" rpy="1.57 1 0" />
+      <!--<origin xyz="-2.0878 -0.58668 0.21577" rpy="1.57 1 0" />-->
+      <origin xyz="-2.0878 -0.58668 0.21577" rpy="0 0 0" />
       <parent link="${prefix}base_link" />
       <child link="${prefix}right_rear_wheel" />
@@ -139,5 +146,6 @@
     </joint>
     <joint name="${prefix}right_front_wheel_joint" type="continuous">
-      <origin xyz="0 -0.58642 0.21577" rpy="1.57 1 0" />
+      <!--<origin xyz="0 -0.58642 0.21577" rpy="1.57 1 0" />-->
+      <origin xyz="0 -0.58642 0.21577" rpy="0 0 0" />
       <parent link="${prefix}base_link" />
       <child link="${prefix}right_front_wheel" />

Commit message: Improved inertias. Still does not rotate fine argh

File: euler_support/urdf/euler_macro.xacro (robot description, xacro)
@@ -6,4 +6,6 @@
 	<xacro:include filename="$(find euler_support)/urdf/eef_macro.xacro" />
 	<xacro:macro name="euler" params="prefix">
+       <property name="base_x_disp" value="1.0438"/>
+       <property name="base_z_disp" value="0.3208"/>
 	<xacro:vetex prefix="vetex_" />
 	<xacro:motoman_mh5lf prefix="motoman_" />
@@ -32,5 +34,5 @@
       <mass value="1.0"/>
       <origin xyz="0 0 0"/>
-      <inertia ixx="0.01" ixy="0.0" ixz="0.0" iyy="0.01" iyz="0.0" izz="0.01"/>
+      <inertia ixx="0.2139" ixy="-0.0026" ixz="-0.04649" iyy="0.3279" iyz="-0.001348" izz="0.1190"/>
     </inertial>
 	</link>
@@ -54,5 +56,5 @@
       <mass value="1.0"/>
       <origin xyz="0 0 0"/>
-      <inertia ixx="0.01" ixy="0.0" ixz="0.0" iyy="0.01" iyz="0.0" izz="0.01"/>
+      <inertia ixx="0.2139" ixy="-0.0026" ixz="-0.04649" iyy="0.3279" iyz="-0.001348" izz="0.1190"/>
     </inertial>
 	</link>
@@ -76,5 +78,5 @@
       <mass value="1.0"/>
       <origin xyz="0 0 0"/>
-      <inertia ixx="0.01" ixy="0.0" ixz="0.0" iyy="0.01" iyz="0.0" izz="0.01"/>
+      <inertia ixx="0.1349" ixy="0.0" ixz="-0.003473" iyy="0.05018" iyz="0.0" izz="0.1454"/>
     </inertial>
 	</link>
@@ -94,7 +96,7 @@
 		</collision>
 		<inertial>
-      <mass value="0.3"/>
+      <mass value="0.250"/>
       <origin xyz="0 0 0"/>
-      <inertia ixx="0.001" ixy="0.0" ixz="0.0" iyy="0.001" iyz="0.0" izz="0.001"/>
+      <inertia ixx="0.0045" ixy="0.0" ixz="0.0" iyy="0.0045" iyz="0.0" izz="0.002048"/>
     </inertial>
 	</link>
@@ -114,7 +116,7 @@
 		</collision>
 		<inertial>
-      <mass value="0.1"/>
+      <mass value="1.20"/>
       <origin xyz="0 0 0"/>
-      <inertia ixx="0.001" ixy="0.0" ixz="0.0" iyy="0.001" iyz="0.0" izz="0.001"/>
+      <inertia ixx="0.002817" ixy="0.0" ixz="0.0" iyy="0.002817" iyz="0.0" izz="0.002347"/>
     </inertial>
 	</link>
@@ -134,7 +136,7 @@
 		</collision>
 		<inertial>
-      <mass value="0.1"/>
+      <mass value="1.20"/>
       <origin xyz="0 0 0"/>
-      <inertia ixx="0.001" ixy="0.0" ixz="0.0" iyy="0.001" iyz="0.0" izz="0.001"/>
+      <inertia ixx="0.002817" ixy="0.0" ixz="0.0" iyy="0.002817" iyz="0.0" izz="0.002347"/>
     </inertial>
 	</link>
@@ -158,7 +160,7 @@
 	</joint>
 	<joint name="${prefix}to_vetex" type="fixed">
-		<parent link="${prefix}base_link" />
-		<child link="${prefix}vetex_base_link" />
-		<origin xyz="0 0 0" rpy="0 0 0" />
+		<parent link="${prefix}vetex_base_link" />
+		<child link="${prefix}base_link" />
+		<origin xyz="${base_x_disp} 0 -${base_z_disp}" rpy="0 0 0" />
 		<axis xyz="0 0 0" />
 	</joint>

File: motoman_mh5lf_support/urdf/mh5lf_macro.xacro (robot description, xacro)
@@ -26,5 +26,5 @@
 		      <mass value="1.0"/>
 		      <origin xyz="0 0 0"/>
-		      <inertia ixx="0.05" ixy="0.0" ixz="0.0" iyy="0.05" iyz="0.0" izz="0.05"/>
+		      <inertia ixx="0.006262" ixy="0.0" ixz="0.0" iyy="0.007306" iyz="0.0" izz="0.005740"/>
 		    </inertial>
 		</link>
@@ -47,5 +47,5 @@
 		      <mass value="1.0"/>
 		      <origin xyz="0 0 0"/>
-		      <inertia ixx="0.05" ixy="0.0" ixz="0.0" iyy="0.05" iyz="0.0" izz="0.05"/>
+		      <inertia ixx="0.00387" ixy="0.0" ixz="-0.00129" iyy="0.005426" iyz="0.0" izz="0.004393"/>
 		    </inertial>
 		</link>
@@ -66,5 +66,5 @@
 		      <mass value="1.0"/>
 		      <origin xyz="0 0 0"/>
-		      <inertia ixx="0.05" ixy="0.0" ixz="0.0" iyy="0.05" iyz="0.0" izz="0.05"/>
+		      <inertia ixx="0.02431" ixy="0.0" ixz="0.0" iyy="0.02190" iyz="0.0" izz="0.005103"/>
 		    </inertial>
 		</link>
@@ -85,5 +85,5 @@
 		      <mass value="1.0"/>
 		      <origin xyz="0 0 0"/>
-		      <inertia ixx="0.05" ixy="0.0" ixz="0.0" iyy="0.05" iyz="0.0" izz="0.05"/>
+		      <inertia ixx="0.002966" ixy="0.0" ixz="0.0" iyy="0.003377" iyz="0.0" izz="0.002966"/>
 		    </inertial>
 		</link>
@@ -104,5 +104,5 @@
 		      <mass value="1.0"/>
 		      <origin xyz="0 0 0"/>
-		      <inertia ixx="0.05" ixy="0.0" ixz="0.0" iyy="0.05" iyz="0.0" izz="0.05"/>
+		      <inertia ixx="0.001861" ixy="0.0" ixz="0.0" iyy="0.010366" iyz="0.0" izz="0.01063"/>
 		    </inertial>
 		</link>
@@ -123,5 +123,5 @@
 		      <mass value="1.0"/>
 		      <origin xyz="0 0 0"/>
-		      <inertia ixx="0.05" ixy="0.0" ixz="0.0" iyy="0.05" iyz="0.0" izz="0.05"/>
+		      <inertia ixx="0.02165" ixy="0.0" ixz="0.0" iyy="0.002165" iyz="0.0" izz="0.002165"/>
 		    </inertial>
 		</link>
@@ -142,5 +142,5 @@
 		      <mass value="1.0"/>
 		      <origin xyz="0 0 0"/>
-		      <inertia ixx="0.05" ixy="0.0" ixz="0.0" iyy="0.05" iyz="0.0" izz="0.05"/>
+		      <inertia ixx="0.02165" ixy="0.0" ixz="0.0" iyy="0.002165" iyz="0.0" izz="0.002165"/>
 		    </inertial>
 		</link>

File: vetex_support/urdf/vetex_macro.xacro (robot description, xacro)
@@ -2,9 +2,11 @@
 <robot xmlns:xacro="http://www.ros.org/wiki/xacro">
   <xacro:macro name="vetex" params="prefix">
+  <property name="base_x_disp" value="1.0438"/>
+  <property name="base_z_disp" value="0.3208"/>
     <!-- link list -->
     <link name="${prefix}base_link">
       <visual>
         <geometry>
-          <mesh filename="package://vetex_support/meshes/visual/base_link.stl" />
+          <mesh filename="package://vetex_support/meshes/collision/base_link_centered.stl" />
         </geometry>
         <material name="euler_gray">
@@ -14,5 +16,5 @@
       <collision>
         <geometry>
-          <mesh filename="package://vetex_support/meshes/visual/base_link.stl" />
+          <mesh filename="package://vetex_support/meshes/collision/base_link_centered.stl" />
         </geometry>
       </collision>
@@ -20,5 +22,5 @@
         <mass value="52.0"/>
         <origin xyz="0 0 0"/>
-        <inertia ixx="1.0" ixy="0.0" ixz="0.0" iyy="1.0" iyz="0.0" izz="1.0"/>
+        <inertia ixx="0.1347" ixy="0.0" ixz="0.0" iyy="0.5214" iyz="0.0" izz="0.6144"/>
       </inertial>
     </link>
@@ -78,5 +80,5 @@
         </visual>
       <collision>
-        <origin xyz="0 0.10 0" rpy="1.5708 0 0" />
+        <origin xyz="0 0. 0" rpy="1.5708 0 0" />
         <!--<origin rpy="3.1415 0 0" />-->
         <geometry>
@@ -117,11 +119,11 @@
     <!-- joint list -->
     <joint name="${prefix}to_footprint" type="fixed">
-      <origin xyz="-1.0439 0 0"/>
-      <parent link="${prefix}base_link" />
-      <child link="${prefix}base_footprint" />
+      <origin xyz="0 0 ${base_z_disp}"/>
+      <parent link="${prefix}base_footprint" />
+      <child link="${prefix}base_link" />
     </joint>
     <joint name="${prefix}left_front_wheel_joint" type="continuous">
       <!--<origin xyz="0 0.58668 0.21577" rpy="1.57 1 0" />-->
-      <origin xyz="0 0.58668 0.21577" rpy="0 0 0" />
+      <origin xyz="${base_x_disp + 0} 0.58668 ${0.21577-base_z_disp}" rpy="0 0 0" />
       <parent link="${prefix}base_link" />
       <child link="${prefix}left_front_wheel" />
@@ -131,5 +133,5 @@
     <joint name="${prefix}left_rear_wheel_joint" type="continuous">
       <!--<origin xyz="-2.0878 0.58642 0.21577" rpy="1.57 1 0" />-->
-      <origin xyz="-2.0878 0.58642 0.21577" rpy="0 0 0" />
+      <origin xyz="${base_x_disp -2.0878} 0.58642 ${0.21577-base_z_disp}" rpy="0 0 0" />
       <parent link="${prefix}base_link" />
       <child link="${prefix}left_rear_wheel" />
@@ -139,5 +141,5 @@
     <joint name="${prefix}right_rear_wheel_joint" type="continuous">
       <!--<origin xyz="-2.0878 -0.58668 0.21577" rpy="1.57 1 0" />-->
-      <origin xyz="-2.0878 -0.58668 0.21577" rpy="0 0 0" />
+      <origin xyz="${base_x_disp -2.0878} -0.58668 ${0.21577-base_z_disp}" rpy="0 0 0" />
       <parent link="${prefix}base_link" />
       <child link="${prefix}right_rear_wheel" />
@@ -147,5 +149,5 @@
     <joint name="${prefix}right_front_wheel_joint" type="continuous">
       <!--<origin xyz="0 -0.58642 0.21577" rpy="1.57 1 0" />-->
-      <origin xyz="0 -0.58642 0.21577" rpy="0 0 0" />
+      <origin xyz="${base_x_disp + 0} -0.58642 ${0.21577 - base_z_disp}" rpy="0 0 0" />
       <parent link="${prefix}base_link" />
       <child link="${prefix}right_front_wheel" />
