Commit message: trying to get this to work in gazebo...

File: vetex_support/urdf/vetex_macro.xacro (robot description, xacro)
@@ -1,114 +1,114 @@
 <?xml version="1.0" ?>
 <robot xmlns:xacro="http://ros.org/wiki/xacro">
-        <xacro:macro name="vetex" params="prefix">
-                <!-- link list -->
-                <link name="${prefix}base_link">
-                        <visual>
-                                <geometry>
-                                        <mesh filename="package://vetex_support/meshes/visual/base_link.stl" />
-                                </geometry>
-                                <material name="euler_gray">
-                                        <color rgba="0.75294 0.75294 0.75294 1" />
-                                </material>
-                        </visual>
-                        <collision>
-                                <geometry>
-                                        <mesh filename="package://vetex_support/meshes/collision/base_link.stl" />
-                                </geometry>
-                        </collision>
-                </link>
-                <link name="${prefix}base_footprint"/>
-                <link name="${prefix}left_front_wheel">
-                        <visual>
-                                <geometry>
-                                        <mesh filename="package://vetex_support/meshes/visual/left_front_wheel.stl" />
-                                </geometry>
-                                <material name="euler_gray"/>
-                        </visual>
-                        <collision>
-                                <geometry>
-                                        <mesh filename="package://vetex_support/meshes/collision/left_front_wheel.stl" />
-                                </geometry>
-                        </collision>
-                </link>
-                <link name="${prefix}left_rear_wheel">
-                        <visual>
-                                <geometry>
-                                        <mesh filename="package://vetex_support/meshes/visual/left_rear_wheel.stl" />
-                                </geometry>
-                                <material name="euler_gray"/>
-                        </visual>
-                        <collision>
-                                <geometry>
-                                        <mesh filename="package://vetex_support/meshes/collision/left_rear_wheel.stl" />
-                                </geometry>
-                        </collision>
-                </link>
-                <link name="${prefix}right_rear_wheel">
-                        <visual>
-                                <origin rpy="3.1415 0 0" />
-                                <geometry>
-                                        <mesh filename="package://vetex_support/meshes/visual/right_rear_wheel.stl" />
-                                </geometry>
-                                <material name="euler_gray"/>
-                                </visual>
-                        <collision>
-                                <origin rpy="3.1415 0 0" />
-                                <geometry>
-                                        <mesh filename="package://vetex_support/meshes/collision/right_rear_wheel.stl" />
-                                </geometry>
-                        </collision>
-                </link>
-                <link name="${prefix}right_front_wheel">
-                        <visual>
-                                <origin rpy="3.1415 0 0" />
-                                <geometry>
-                                        <mesh filename="package://vetex_support/meshes/visual/right_front_wheel.stl" />
-                                </geometry>
-                                <material name="euler_gray"/>
-                        </visual>
-                        <collision>
-                                <origin rpy="3.1415 0 0" />
-                                <geometry>
-                                        <mesh filename="package://vetex_support/meshes/collision/right_front_wheel.stl" />
-                                </geometry>
-                        </collision>
-                </link>
-                <!-- end of link list -->
-                <!-- joint list -->
-                <joint name="${prefix}to_footprint" type="fixed">
-                    <origin xyz="-1.0439 0 0"/>
-                    <parent link="${prefix}base_link" />
-                    <child link="${prefix}base_footprint" />
-                </joint>
-                <joint name="${prefix}left_front_wheel" type="continuous">
-                        <origin xyz="0 0.58668 0.21577" rpy="0 1 0" />
-                        <parent link="${prefix}base_link" />
-                        <child link="${prefix}left_front_wheel" />
-                        <axis xyz="0 1 0" />
-                        <limit effort="0" velocity="3" />
-                </joint>
-                <joint name="${prefix}left_rear_wheel" type="continuous">
-                        <origin xyz="-2.0878 0.58642 0.21577" rpy="0 1 0" />
-                        <parent link="${prefix}base_link" />
-                        <child link="${prefix}left_rear_wheel" />
-                        <axis xyz="0 1 0" />
-                        <limit effort="0" velocity="3" />
-                </joint>
-                <joint name="${prefix}right_rear_wheel" type="continuous">
-                        <origin xyz="-2.0878 -0.58668 0.21577" rpy="0 1 0" />
-                        <parent link="${prefix}base_link" />
-                        <child link="${prefix}right_rear_wheel" />
-                        <axis xyz="0 1 0" />
-                        <limit effort="0" velocity="3" />
-                </joint>
-                <joint name="${prefix}right_front_wheel" type="continuous">
-                        <origin xyz="0 -0.58642 0.21577" rpy="0 0 0" />
-                        <parent link="${prefix}base_link" />
-                        <child link="${prefix}right_front_wheel" />
-                        <axis xyz="0 1 0" />
-                        <limit effort="0" velocity="3" />
-                </joint>
-               	<!-- end of joint list -->
-        </xacro:macro>
+  <xacro:macro name="vetex" params="prefix">
+    <!-- link list -->
+    <link name="${prefix}base_link">
+      <visual>
+        <geometry>
+          <mesh filename="package://vetex_support/meshes/visual/base_link.stl" />
+        </geometry>
+        <material name="euler_gray">
+          <color rgba="0.75294 0.75294 0.75294 1" />
+        </material>
+      </visual>
+      <collision>
+        <geometry>
+          <mesh filename="package://vetex_support/meshes/collision/base_link.stl" />
+        </geometry>
+      </collision>
+    </link>
+    <link name="${prefix}base_footprint"/>
+    <link name="${prefix}left_front_wheel">
+      <visual>
+        <geometry>
+          <mesh filename="package://vetex_support/meshes/visual/left_front_wheel.stl" />
+        </geometry>
+        <material name="euler_gray"/>
+      </visual>
+      <collision>
+        <geometry>
+          <mesh filename="package://vetex_support/meshes/collision/left_front_wheel.stl" />
+        </geometry>
+      </collision>
+    </link>
+    <link name="${prefix}left_rear_wheel">
+      <visual>
+        <geometry>
+          <mesh filename="package://vetex_support/meshes/visual/left_rear_wheel.stl" />
+        </geometry>
+        <material name="euler_gray"/>
+      </visual>
+      <collision>
+        <geometry>
+          <mesh filename="package://vetex_support/meshes/collision/left_rear_wheel.stl" />
+        </geometry>
+      </collision>
+    </link>
+    <link name="${prefix}right_rear_wheel">
+      <visual>
+        <origin rpy="3.1415 0 0" />
+        <geometry>
+          <mesh filename="package://vetex_support/meshes/visual/right_rear_wheel.stl" />
+        </geometry>
+        <material name="euler_gray"/>
+        </visual>
+      <collision>
+        <origin rpy="3.1415 0 0" />
+        <geometry>
+          <mesh filename="package://vetex_support/meshes/collision/right_rear_wheel.stl" />
+        </geometry>
+      </collision>
+    </link>
+    <link name="${prefix}right_front_wheel">
+      <visual>
+        <origin rpy="3.1415 0 0" />
+        <geometry>
+          <mesh filename="package://vetex_support/meshes/visual/right_front_wheel.stl" />
+        </geometry>
+        <material name="euler_gray"/>
+      </visual>
+      <collision>
+        <origin rpy="3.1415 0 0" />
+        <geometry>
+          <mesh filename="package://vetex_support/meshes/collision/right_front_wheel.stl" />
+        </geometry>
+      </collision>
+    </link>
+    <!-- end of link list -->
+    <!-- joint list -->
+    <joint name="${prefix}to_footprint" type="fixed">
+      <origin xyz="-1.0439 0 0"/>
+      <parent link="${prefix}base_link" />
+      <child link="${prefix}base_footprint" />
+    </joint>
+    <joint name="${prefix}left_front_wheel_joint" type="continuous">
+      <origin xyz="0 0.58668 0.21577" rpy="0 1 0" />
+      <parent link="${prefix}base_link" />
+      <child link="${prefix}left_front_wheel" />
+      <axis xyz="0 1 0" />
+      <limit effort="0" velocity="3" />
+    </joint>
+    <joint name="${prefix}left_rear_wheel_joint" type="continuous">
+      <origin xyz="-2.0878 0.58642 0.21577" rpy="0 1 0" />
+      <parent link="${prefix}base_link" />
+      <child link="${prefix}left_rear_wheel" />
+      <axis xyz="0 1 0" />
+      <limit effort="0" velocity="3" />
+    </joint>
+    <joint name="${prefix}right_rear_wheel_joint" type="continuous">
+      <origin xyz="-2.0878 -0.58668 0.21577" rpy="0 1 0" />
+      <parent link="${prefix}base_link" />
+      <child link="${prefix}right_rear_wheel" />
+      <axis xyz="0 1 0" />
+      <limit effort="0" velocity="3" />
+    </joint>
+    <joint name="${prefix}right_front_wheel_joint" type="continuous">
+      <origin xyz="0 -0.58642 0.21577" rpy="0 0 0" />
+      <parent link="${prefix}base_link" />
+      <child link="${prefix}right_front_wheel" />
+      <axis xyz="0 1 0" />
+      <limit effort="0" velocity="3" />
+    </joint>
+    <!-- end of joint list -->
+  </xacro:macro>
 </robot>

Commit message: Fixed displacements for rgb and depth frame to be in Y now

File: euler_support/urdf/asus_xtion_pro.xacro (robot description, xacro)
@@ -27,5 +27,5 @@
   </joint>
   <joint name="${sensor_name}_depth_joint" type="fixed">
-    <origin xyz="0.049 0 0" rpy="-1.5708 0 -1.5708" />
+    <origin xyz="0 -0.049 0" rpy="-1.5708 0 -1.5708" />
     <parent link="${sensor_name}_bodycenter" />
     <child link="${sensor_name}_depth_frame" />
@@ -33,5 +33,5 @@
   <link name="${sensor_name}_depth_frame" />
   <joint name="${sensor_name}_rgb_joint" type="fixed">
-    <origin xyz="0.022 0 0" rpy="-1.5708 0 -1.5708" />
+    <origin xyz="0 -0.022 0" rpy="-1.5708 0 -1.5708" />
     <parent link="${sensor_name}_bodycenter" />
     <child link="${sensor_name}_rgb_frame" />
