Commit message: Added changes over New Year

File: euler_gazebo/urdf/euler.gazebo.components.xacro (robot description, xacro)
@@ -4,5 +4,5 @@
   <xacro:include filename="$(find euler_gazebo)/urdf/euler.gazebo.component_macros.xacro"/>
   <xacro:euler prefix=""/>
-  <euler_arm prefix=""/>
+  <!--<euler_arm prefix=""/>-->
   <euler_base prefix="" side="left"/>
   <euler_base prefix="" side="right"/>

File: euler_gazebo/urdf/euler_gazebo.xacro (robot description, xacro)
@@ -4,5 +4,5 @@
   <xacro:include filename="$(find euler_gazebo)/urdf/euler.gazebo.components.xacro"/>
   <xacro:include filename="$(find euler_gazebo)/urdf/euler.gazebo.controllers.xacro"/>
-  <gazebo reference="frame_left">
+<!--  <gazebo reference="frame_left">
     <material>Gazebo/Grey</material>
   </gazebo>
@@ -13,7 +13,9 @@
     <material>Gazebo/Grey</material>
   </gazebo>
+-->
   <gazebo reference="vetex_base_link">
     <material>Gazebo/Grey</material>
   </gazebo>
+<!--
   <gazebo reference="motoman_base_link">
     <material>Gazebo/Blue</material>
@@ -46,31 +48,28 @@
     <material>Gazebo/Yellow</material>
   </gazebo>
+-->
   <gazebo reference="vetex_right_rear_wheel">
     <material>Gazebo/Black</material>
-    <mu1 value="1.0" />
-    <mu2 value="1.0" />
-    <kp value="10000000.0" />
-    <kd value="1.0" />
+    <mu1 value="0.9" />
+    <mu2 value="0.9" />
+    <minDepth>0.0001</minDepth>
   </gazebo>
   <gazebo reference="vetex_right_front_wheel">
     <material>Gazebo/Black</material>
-    <mu1 value="1.0" />
-    <mu2 value="1.0" />
-    <kp value="10000000.0" />
-    <kd value="1.0" />
+    <mu1 value="0.9" />
+    <mu2 value="0.9" />
+    <minDepth>0.0001</minDepth>
   </gazebo>
   <gazebo reference="vetex_left_rear_wheel">
     <material>Gazebo/Black</material>
-    <mu1 value="1.0" />
-    <mu2 value="1.0" />
-    <kp value="10000000.0" />
-    <kd value="1.0" />
+    <mu1 value="0.9" />
+    <mu2 value="0.9" />
+    <minDepth>0.001</minDepth>
   </gazebo>
   <gazebo reference="vetex_left_front_wheel">
     <material>Gazebo/Black</material>
-    <mu1 value="1.0" />
-    <mu2 value="1.0" />
-    <kp value="10000000.0" />
-    <kd value="1.0" />
+    <mu1 value="0.9" />
+    <mu2 value="0.9" />
+    <minDepth>0.0001</minDepth>
   </gazebo>
 </robot>

File: euler_support/urdf/euler_macro.xacro (robot description, xacro)
@@ -1,5 +1,5 @@
 <?xml version="1.0" ?>
 <robot xmlns:xacro="http://www.ros.org/wiki/xacro">
-	<xacro:include filename="$(find vetex_support)/urdf/vetex_macro.xacro" />
+	<xacro:include filename="$(find vetex_support)/urdf/vetex_test_macro.xacro" />
 	<xacro:include filename="$(find motoman_mh5lf_support)/urdf/mh5lf_macro.xacro" />
 	<xacro:include filename="$(find euler_support)/urdf/asus_xtion_pro.xacro" />
@@ -7,11 +7,11 @@
 	<xacro:macro name="euler" params="prefix">
 	<xacro:vetex prefix="vetex_" />
-	<xacro:motoman_mh5lf prefix="motoman_" />
+	<!--<xacro:motoman_mh5lf prefix="motoman_" />-->
 	<!-- <xacro:asus_xtion_pro sensor_name="" off_x="0.461" off_y="0" off_z="2.103" off_rr="1.5708" off_rp="1.8849" off_ry="0"/>        -->
-	<xacro:eef prefix=""/>
+	<!--<xacro:eef prefix=""/>         -->
 	<!--link list -->
-	<link name="${prefix}base_link">
-	</link>
-	<link name="${prefix}frame_left">
+	<!--<link name="${prefix}base_link">
+	</link> -->
+	<!--<link name="${prefix}frame_left">
 		<visual>
 			<origin xyz="0 0 0" rpy="0 0 0" />
@@ -157,10 +157,11 @@
 		<axis xyz="0 0 0" />
 	</joint>
-	<joint name="${prefix}to_vetex" type="fixed">
+	 -->
+	<!--<joint name="${prefix}to_vetex" type="fixed">
 		<parent link="${prefix}base_link" />
 		<child link="${prefix}vetex_base_link" />
 		<origin xyz="0 0 0" rpy="0 0 0" />
 		<axis xyz="0 0 0" />
-	</joint>
+	</joint>--> <!--
 	<joint name="${prefix}to_arm" type="fixed">
 		<parent link="${prefix}base_link" />
@@ -192,4 +193,5 @@
 		<origin xyz="0.098 0 0" rpy="0 1.57 0" />
 	</joint>
+-->
 </xacro:macro>
 </robot>

File: vetex_support/urdf/vetex_test_macro.xacro (robot description, xacro)
@@ -6,5 +6,5 @@
       <visual>
         <geometry>
-          <mesh filename="package://vetex_support/meshes/visual/base_link.stl" />
+          <mesh filename="package://vetex_support/meshes/visual/test_base.stl" />
         </geometry>
         <material name="euler_gray">
@@ -14,11 +14,11 @@
       <collision>
         <geometry>
-          <mesh filename="package://vetex_support/meshes/collision/base_link_03.stl" />
+          <mesh filename="package://vetex_support/meshes/visual/test_base.stl" />
         </geometry>
       </collision>
       <inertial>
-        <mass value="52.0"/>
-        <origin xyz="-1.19 0 0.19"/>
-        <inertia ixx="0.1347" ixy="0.0" ixz="0.0" iyy="0.5214" iyz="0.0" izz="0.6144"/>
+        <mass value="20.0"/>
+        <origin xyz="0 0 0"/>
+        <inertia ixx="0.07" ixy="0.0" ixz="0.0" iyy="0.5433" iyz="0.0" izz="0.569"/>
       </inertial>
     </link>
@@ -27,5 +27,5 @@
       <visual>
         <geometry>
-          <mesh filename="package://vetex_support/meshes/visual/left_front_wheel.stl" />
+          <mesh filename="package://vetex_support/meshes/visual/test_wheel_015.stl" />
         </geometry>
         <material name="euler_black">
@@ -35,11 +35,11 @@
       <collision>
         <geometry>
-          <mesh filename="package://vetex_support/meshes/collision/left_front_wheel_02.stl" />
+          <mesh filename="package://vetex_support/meshes/visual/test_wheel_015.stl" />
         </geometry>
       </collision>
       <inertial>
-        <mass value="4.0"/>
-        <origin xyz="0 -0.13 0"/>
-        <inertia ixx="0.0139" ixy="0.0" ixz="0.0" iyy="0.01818" iyz="0.0" izz="0.0139"/>
+        <mass value="2.0"/>
+        <origin xyz="0 0 0"/>
+        <inertia ixx="0.0126" ixy="0.0" ixz="0.0" iyy="0.0206" iyz="0.0" izz="0.0126"/>
       </inertial>
     </link>
@@ -47,6 +47,5 @@
       <visual>
         <geometry>
-          <!--<cylinder length="0.2" radius="0.2"/>-->
-          <mesh filename="package://vetex_support/meshes/visual/left_rear_wheel.stl" />
+          <mesh filename="package://vetex_support/meshes/visual/test_wheel_015.stl" />
         </geometry>
         <material name="euler_black"/>
@@ -56,11 +55,11 @@
         <geometry>
           <!-- <cylinder length="0.2" radius="0.2"/>-->
-          <mesh filename="package://vetex_support/meshes/collision/left_rear_wheel_02.stl" />
+          <mesh filename="package://vetex_support/meshes/visual/test_wheel_015.stl" />
         </geometry>
       </collision>
       <inertial>
-        <mass value="4.0"/>
-        <origin xyz="0 -0.15 0"/>
-        <inertia ixx="0.01292" ixy="0.0" ixz="0.0" iyy="0.02012" iyz="0.0" izz="0.01292"/>
+        <mass value="2.0"/>
+        <origin xyz="0 0 0"/>
+        <inertia ixx="0.0126" ixy="0.0" ixz="0.0" iyy="0.0206" iyz="0.0" izz="0.0126"/>
       </inertial>
     </link>
@@ -69,20 +68,19 @@
         <origin rpy="3.1415 0 0" />
         <geometry>
-          <mesh filename="package://vetex_support/meshes/visual/right_rear_wheel.stl" />
+          <mesh filename="package://vetex_support/meshes/visual/test_wheel_015.stl" />
         </geometry>
         <material name="euler_black"/>
         </visual>
       <collision>
-        <!--<origin xyz="0 0.10 0" rpy="1.5708 0 0" />-->
         <origin rpy="3.1415 0 0" />
         <geometry>
           <!--<cylinder length="0.2" radius="0.2"/>-->
-          <mesh filename="package://vetex_support/meshes/collision/right_rear_wheel_02.stl" />
+          <mesh filename="package://vetex_support/meshes/visual/test_wheel_015.stl" />
         </geometry>
       </collision>
       <inertial>
-        <mass value="4.0"/>
-        <origin xyz="0 0.13 0"/>
-        <inertia ixx="0.0139" ixy="0.0" ixz="0.0" iyy="0.01818" iyz="0.0" izz="0.0139"/>
+        <mass value="2.0"/>
+        <origin xyz="0 0 0"/>
+        <inertia ixx="0.0126" ixy="0.0" ixz="0.0" iyy="0.0206" iyz="0.0" izz="0.0126"/>
       </inertial>
     </link>
@@ -91,6 +89,5 @@
         <origin rpy="3.1415 0 0" />
         <geometry>
-          <!--<cylinder length="0.2" radius="0.2"/>-->
-          <mesh filename="package://vetex_support/meshes/visual/right_front_wheel.stl" />
+          <mesh filename="package://vetex_support/meshes/visual/test_wheel_015.stl" />
         </geometry>
         <material name="euler_black"/>
@@ -99,51 +96,47 @@
         <origin rpy="3.1415 0 0" />
         <geometry>
-          <mesh filename="package://vetex_support/meshes/collision/right_front_wheel_02.stl" />
+          <mesh filename="package://vetex_support/meshes/visual/test_wheel_015.stl" />
         </geometry>
       </collision>
       <inertial>
-        <mass value="4.0"/>
-        <origin xyz="0 0.15 0"/>
-        <inertia ixx="0.01292" ixy="0.0" ixz="0.0" iyy="0.02012" iyz="0.0" izz="0.01292"/>
+        <mass value="2.0"/>
+        <origin xyz="0 0 0"/>
+        <inertia ixx="0.0126" ixy="0.0" ixz="0.0" iyy="0.0206" iyz="0.0" izz="0.0126"/>
       </inertial>
     </link>
     <!-- end of link list -->
     <!-- joint list -->
-    <joint name="${prefix}to_footprint" type="fixed">
-      <origin xyz="-1.0439 0 0"/>
-      <parent link="${prefix}base_link" />
-      <child link="${prefix}base_footprint" />
+    <joint name="${prefix}to_base_link" type="fixed">
+      <origin xyz="0 0 0.31"/>
+      <parent link="${prefix}base_footprint" />
+      <child link="${prefix}base_link" />
     </joint>
     <joint name="${prefix}left_front_wheel_joint" type="continuous">
-      <!--<origin xyz="0 0.58668 0.21577" rpy="1.57 1 0" />-->
-      <origin xyz="0 0.58668 0.21577" rpy="0 0 0" />
+      <origin xyz="1.0 0.52 -0.10" rpy="0 0 0" />
       <parent link="${prefix}base_link" />
       <child link="${prefix}left_front_wheel" />
       <axis xyz="0 1 0" />
-      <limit effort="100" velocity="3" />
+      <limit effort="100" velocity="10" />
     </joint>
     <joint name="${prefix}left_rear_wheel_joint" type="continuous">
-      <!--<origin xyz="-2.0878 0.58642 0.21577" rpy="1.57 1 0" />-->
-      <origin xyz="-2.0878 0.58642 0.21577" rpy="0 0 0" />
+      <origin xyz="-1.0 0.52 -0.10" rpy="0 0 0" />
       <parent link="${prefix}base_link" />
       <child link="${prefix}left_rear_wheel" />
       <axis xyz="0 1 0" />
-      <limit effort="100" velocity="3" />
+      <limit effort="100" velocity="10" />
     </joint>
     <joint name="${prefix}right_rear_wheel_joint" type="continuous">
-      <!--<origin xyz="-2.0878 -0.58668 0.21577" rpy="1.57 1 0" />-->
-      <origin xyz="-2.0878 -0.58668 0.21577" rpy="0 0 0" />
+      <origin xyz="-1.0 -0.52 -0.10" rpy="0 0 0" />
       <parent link="${prefix}base_link" />
       <child link="${prefix}right_rear_wheel" />
       <axis xyz="0 1 0" />
-      <limit effort="100" velocity="3" />
+      <limit effort="100" velocity="10" />
     </joint>
     <joint name="${prefix}right_front_wheel_joint" type="continuous">
-      <!--<origin xyz="0 -0.58642 0.21577" rpy="1.57 1 0" />-->
-      <origin xyz="0 -0.58642 0.21577" rpy="0 0 0" />
+      <origin xyz="1.0 -0.52 -0.10" rpy="0 0 0" />
       <parent link="${prefix}base_link" />
       <child link="${prefix}right_front_wheel" />
       <axis xyz="0 1 0" />
-      <limit effort="100" velocity="3" />
+      <limit effort="100" velocity="10" />
     </joint>
     <!-- end of joint list -->
