Commit message: some xacro cleanup. still not working

File: euler_gazebo/urdf/euler.gazebo.component_macros.xacro (robot description, xacro)
@@ -1,7 +1,13 @@
 <?xml version="1.0"?>
-<robot xmlns:xacro="http://www.ros.org/wiki/xacro">
+<robot  xmlns:xacro="http://www.ros.org/wiki/xacro">
+<!-- <robot
+    xmlns:controller="http://playerstage.sourceforge.net/gazebo/xmlschema/#controller"
+    xmlns:interface="http://playerstage.sourceforge.net/gazebo/xmlschema/#interface"
+    xmlns:sensor="http://playerstage.sourceforge.net/gazebo/xmlschema/#sensor"
+    xmlns:xacro="http://playerstage.sourceforge.net/gazebo/xmlschema/#interface">
+ -->
   <!-- link xacro -->
   <xacro:macro name="gazebo_link" params="prefix link_name gravity_off static collide">
-    <gazebo reference="${prefix}${link_name}_link">
+    <gazebo reference="${prefix}${link_name}">
       <selfCollide>${collide}</selfCollide>
       <static>${static}</static>
@@ -79,10 +85,10 @@
     <gazebo_joint prefix="${prefix}" joint_name="motoman_joint_b" kd="4" kp="10"/>
     <gazebo_joint prefix="${prefix}" joint_name="motoman_joint_t" kd="4" kp="10"/>
-    <gazebo_simple_pos_trans prefix="${prefix}" joint_name="motoman_joint_s_joint" reduction="1" tc="1"/>
-    <gazebo_simple_pos_trans prefix="${prefix}" joint_name="motoman_joint_l_joint" reduction="1" tc="1"/>
-    <gazebo_simple_pos_trans prefix="${prefix}" joint_name="motoman_joint_u_joint" reduction="1" tc="1"/>
-    <gazebo_simple_pos_trans prefix="${prefix}" joint_name="motoman_joint_r_joint" reduction="1" tc="1"/>
-    <gazebo_simple_pos_trans prefix="${prefix}" joint_name="motoman_joint_b_joint" reduction="1" tc="1"/>
-    <gazebo_simple_pos_trans prefix="${prefix}" joint_name="motoman_joint_t_joint" reduction="1" tc="1"/>
+    <gazebo_simple_pos_trans prefix="${prefix}" joint_name="motoman_joint_s" reduction="1" tc="1"/>
+    <gazebo_simple_pos_trans prefix="${prefix}" joint_name="motoman_joint_l" reduction="1" tc="1"/>
+    <gazebo_simple_pos_trans prefix="${prefix}" joint_name="motoman_joint_u" reduction="1" tc="1"/>
+    <gazebo_simple_pos_trans prefix="${prefix}" joint_name="motoman_joint_r" reduction="1" tc="1"/>
+    <gazebo_simple_pos_trans prefix="${prefix}" joint_name="motoman_joint_b" reduction="1" tc="1"/>
+    <gazebo_simple_pos_trans prefix="${prefix}" joint_name="motoman_joint_t" reduction="1" tc="1"/>
   </xacro:macro>
   <!-- euler kinect xacro -->

File: euler_gazebo/urdf/euler_gazebo.xacro (robot description, xacro)
@@ -1,16 +1,6 @@
 <?xml version="1.0" ?>
-<robot name="euler" xmlns:xacro="http://www.ros.org/wiki/xacro">
-  <xacro:property name="robot_name" value="euler" />
+  <robot name="euler" xmlns:xacro="http://www.ros.org/wiki/xacro">
   <xacro:include filename="$(find euler_support)/urdf/euler_macro.xacro" />
-  <xacro:include filename="$(find euler_gazebo)/urdf/euler.gazebo.component_macros.xacro"/>
-  <xacro:euler prefix=""/>
-  <euler_base prefix="" side="left"/>
-  <euler_base prefix="" side="right"/>
-  <euler_arm prefix=""/>
-  <gazebo>
-    <plugin name="gazebo_ros_control" filename="libgazebo_ros_control.so">
-      <robotNamespace>${robot_name}</robotNamespace>
-      <robotSimType>gazebo_ros_control/DefaultRobotHWSim</robotSimType>
-    </plugin>
-  </gazebo>
+  <xacro:include filename="$(find euler_gazebo)/urdf/euler.gazebo.components.xacro"/>
+  <xacro:include filename="$(find euler_gazebo)/urdf/euler.gazebo.controllers.xacro"/>
 </robot>

File: euler_support/urdf/asus_xtion_pro.xacro (robot description, xacro)
@@ -1,4 +1,5 @@
 <?xml version="1.0"?>
-<robot xmlns:xacro="http://ros.org/wiki/xacro">
+<!-- <robot xmlns:xacro="http://ros.org/wiki/xacro"> -->
+<robot  xmlns:xacro="http://www.ros.org/wiki/xacro">
 <xacro:macro name="asus_xtion_pro" params="sensor_name off_x off_y off_z off_rr off_rp off_ry">
   <xacro:property name="M_PI" value="3.14159"/>

File: euler_support/urdf/eef_macro.xacro (robot description, xacro)
@@ -1,4 +1,6 @@
 <?xml version="1.0" ?>
-<robot xmlns:xacro="http://ros.org/wiki/xacro">
+<robot  xmlns:xacro="http://www.ros.org/wiki/xacro">
+<!-- <robot xmlns:xacro="http://ros.org/wiki/xacro">
+ -->
   <xacro:macro name="eef" params="prefix">
     <material name="eef_color">

File: euler_support/urdf/euler_macro.xacro (robot description, xacro)
@@ -1,9 +1,9 @@
 <?xml version="1.0" ?>
-<robot xmlns:xacro="http://ros.org/wiki/xacro">
-<xacro:include filename="$(find vetex_support)/urdf/vetex_macro.xacro" />
-<xacro:include filename="$(find motoman_mh5lf_support)/urdf/mh5lf_macro.xacro" />
-<xacro:include filename="$(find euler_support)/urdf/asus_xtion_pro.xacro" />
-<xacro:include filename="$(find euler_support)/urdf/eef_macro.xacro" />
-<xacro:macro name="euler" params="prefix">
+<robot xmlns:xacro="http://www.ros.org/wiki/xacro">
+	<xacro:include filename="$(find vetex_support)/urdf/vetex_macro.xacro" />
+	<xacro:include filename="$(find motoman_mh5lf_support)/urdf/mh5lf_macro.xacro" />
+	<xacro:include filename="$(find euler_support)/urdf/asus_xtion_pro.xacro" />
+	<xacro:include filename="$(find euler_support)/urdf/eef_macro.xacro" />
+	<xacro:macro name="euler" params="prefix">
 	<xacro:vetex prefix="vetex_" />
 	<xacro:motoman_mh5lf prefix="motoman_" />
@@ -12,5 +12,5 @@
 	<!--link list -->
 	<link name="${prefix}base_link"> </link>
-  <link name="${prefix}frame_left">
+	<link name="${prefix}frame_left">
 		<visual>
 			<origin xyz="0 0 0" rpy="0 0 0" />

File: motoman_mh5lf_support/urdf/mh5lf_macro.xacro (robot description, xacro)
@@ -1,4 +1,5 @@
 <?xml version="1.0" ?>
-<robot xmlns:xacro="http://ros.org/wiki/xacro">
+<!-- <robot xmlns:xacro="http://ros.org/wiki/xacro"> -->
+<robot	xmlns:xacro="http://www.ros.org/wiki/xacro">
 	<xacro:macro name="motoman_mh5lf" params="prefix">
 		<!-- link list -->

File: vetex_support/urdf/vetex_macro.xacro (robot description, xacro)
@@ -1,4 +1,4 @@
 <?xml version="1.0" ?>
-<robot xmlns:xacro="http://ros.org/wiki/xacro">
+<robot xmlns:xacro="http://www.ros.org/wiki/xacro">
   <xacro:macro name="vetex" params="prefix">
     <!-- link list -->

Commit message: basic running version in gazebo. havent tried any craftsman stuff yet

File: euler_gazebo/urdf/euler.gazebo.component_macros.xacro (robot description, xacro)
@@ -66,10 +66,8 @@
     <gazebo_joint prefix="${prefix}" joint_name="vetex_${side}_front_wheel_joint" kd="4" kp="10"/>
     <gazebo_joint prefix="${prefix}" joint_name="vetex_${side}_rear_wheel_joint" kd="4" kp="10"/>
-<!--     <gazebo_dif_drive_trans prefix="${robot_name}/${side}" joint_name="wheel" reduction="1" tc="1"/>
- -->
     <gazebo_dif_drive_trans prefix="${prefix}" joint_name="vetex_${side}_front_wheel" reduction="1" tc="1"/>
     <gazebo_dif_drive_trans prefix="${prefix}" joint_name="vetex_${side}_rear_wheel"  reduction="1" tc="1"/>
   </xacro:macro>
-  <!-- tracbot arm xacro -->
+  <!-- euler arm xacro -->
   <xacro:macro name="euler_arm" params="prefix">
     <gazebo_link prefix="${prefix}" link_name="motoman_link_s" collide="true" static="true" gravity_off="true"/>

File: euler_gazebo/urdf/euler.gazebo.components.xacro (robot description, xacro)
@@ -5,3 +5,5 @@
   <xacro:euler prefix=""/>
   <euler_arm prefix=""/>
+  <euler_base prefix="" side="left"/>
+  <euler_base prefix="" side="right"/>
 </robot>

File: euler_gazebo/urdf/euler.gazebo.controllers.xacro (robot description, xacro)
@@ -1,8 +1,4 @@
 <?xml version="1.0"?>
 <robot	xmlns:xacro="http://www.ros.org/wiki/xacro">
-<!-- <robot xmlns:controller="http://playerstage.sourceforge.net/gazebo/xmlschema/#controller"
-			xmlns:interface="http://playerstage.sourceforge.net/gazebo/xmlschema/#interface"
-			xmlns:sensor="http://playerstage.sourceforge.net/gazebo/xmlschema/#sensor"
-			xmlns:xacro="http://playerstage.sourceforge.net/gazebo/xmlschema/#interface"> -->
   <gazebo>
     <plugin name="gazebo_ros_control" filename="libgazebo_ros_control.so">

File: euler_support/urdf/euler_macro.xacro (robot description, xacro)
@@ -8,8 +8,9 @@
 	<xacro:vetex prefix="vetex_" />
 	<xacro:motoman_mh5lf prefix="motoman_" />
-	<xacro:asus_xtion_pro sensor_name="" off_x="0.461" off_y="0" off_z="2.103" off_rr="1.5708" off_rp="1.8849" off_ry="0"/>
+	<!-- <xacro:asus_xtion_pro sensor_name="" off_x="0.461" off_y="0" off_z="2.103" off_rr="1.5708" off_rp="1.8849" off_ry="0"/>        -->
 	<xacro:eef prefix=""/>
 	<!--link list -->
-	<link name="${prefix}base_link"> </link>
+	<link name="${prefix}base_link">
+	</link>
 	<link name="${prefix}frame_left">
 		<visual>
@@ -28,4 +29,9 @@
 			</geometry>
 		</collision>
+		<inertial>
+      <mass value="0.1"/>
+      <origin xyz="0 0 0"/>
+      <inertia ixx="1.0" ixy="0.0" ixz="0.0" iyy="1.0" iyz="0.0" izz="1.0"/>
+    </inertial>
 	</link>
 	<link name="${prefix}frame_right">
@@ -45,4 +51,9 @@
 			</geometry>
 		</collision>
+		<inertial>
+      <mass value="0.1"/>
+      <origin xyz="0 0 0"/>
+      <inertia ixx="1.0" ixy="0.0" ixz="0.0" iyy="1.0" iyz="0.0" izz="1.0"/>
+    </inertial>
 	</link>
 	<link name="${prefix}frame_top">
@@ -62,4 +73,9 @@
 			</geometry>
 		</collision>
+		<inertial>
+      <mass value="0.1"/>
+      <origin xyz="0 0 0"/>
+      <inertia ixx="1.0" ixy="0.0" ixz="0.0" iyy="1.0" iyz="0.0" izz="1.0"/>
+    </inertial>
 	</link>
 	<link name="${prefix}sick_nav350">
@@ -77,4 +93,9 @@
 			</geometry>
 		</collision>
+		<inertial>
+      <mass value="0.1"/>
+      <origin xyz="0 0 0"/>
+      <inertia ixx="1.0" ixy="0.0" ixz="0.0" iyy="1.0" iyz="0.0" izz="1.0"/>
+    </inertial>
 	</link>
 	<link name="${prefix}front_sick_s300">
@@ -92,4 +113,9 @@
 			</geometry>
 		</collision>
+		<inertial>
+      <mass value="0.1"/>
+      <origin xyz="0 0 0"/>
+      <inertia ixx="1.0" ixy="0.0" ixz="0.0" iyy="1.0" iyz="0.0" izz="1.0"/>
+    </inertial>
 	</link>
 	<link name="${prefix}rear_sick_s300">
@@ -107,4 +133,9 @@
 			</geometry>
 		</collision>
+		<inertial>
+      <mass value="0.1"/>
+      <origin xyz="0 0 0"/>
+      <inertia ixx="1.0" ixy="0.0" ixz="0.0" iyy="1.0" iyz="0.0" izz="1.0"/>
+    </inertial>
 	</link>
 	<joint name="${prefix}frame_left" type="fixed" >

File: motoman_mh5lf_support/urdf/mh5lf_macro.xacro (robot description, xacro)
@@ -23,4 +23,9 @@
 				</material>
 			</collision>
+			<inertial>
+		      <mass value="0.1"/>
+		      <origin xyz="0 0 0"/>
+		      <inertia ixx="1.0" ixy="0.0" ixz="0.0" iyy="1.0" iyz="0.0" izz="1.0"/>
+		    </inertial>
 		</link>
 		<link name="${prefix}link_s">
@@ -39,4 +44,9 @@
 				<material name="yellow"/>
 			</collision>
+			<inertial>
+		      <mass value="0.1"/>
+		      <origin xyz="0 0 0"/>
+		      <inertia ixx="1.0" ixy="0.0" ixz="0.0" iyy="1.0" iyz="0.0" izz="1.0"/>
+		    </inertial>
 		</link>
 		<link name="${prefix}link_l">
@@ -53,4 +63,9 @@
 				<material name="yellow"/>
 			</collision>
+			<inertial>
+		      <mass value="0.1"/>
+		      <origin xyz="0 0 0"/>
+		      <inertia ixx="1.0" ixy="0.0" ixz="0.0" iyy="1.0" iyz="0.0" izz="1.0"/>
+		    </inertial>
 		</link>
 		<link name="${prefix}link_u">
@@ -67,4 +82,9 @@
 				<material name="yellow"/>
 			</collision>
+			<inertial>
+		      <mass value="0.1"/>
+		      <origin xyz="0 0 0"/>
+		      <inertia ixx="1.0" ixy="0.0" ixz="0.0" iyy="1.0" iyz="0.0" izz="1.0"/>
+		    </inertial>
 		</link>
 		<link name="${prefix}link_r">
@@ -81,4 +101,9 @@
 				<material name="yellow"/>
 			</collision>
+			<inertial>
+		      <mass value="0.1"/>
+		      <origin xyz="0 0 0"/>
+		      <inertia ixx="1.0" ixy="0.0" ixz="0.0" iyy="1.0" iyz="0.0" izz="1.0"/>
+		    </inertial>
 		</link>
 		<link name="${prefix}link_b">
@@ -95,4 +120,9 @@
 				<material name="yellow"/>
 			</collision>
+			<inertial>
+		      <mass value="0.1"/>
+		      <origin xyz="0 0 0"/>
+		      <inertia ixx="1.0" ixy="0.0" ixz="0.0" iyy="1.0" iyz="0.0" izz="1.0"/>
+		    </inertial>
 		</link>
 		<link name="${prefix}link_t">
@@ -109,4 +139,9 @@
 				<material name="yellow"/>
 			</collision>
+			<inertial>
+		      <mass value="0.1"/>
+		      <origin xyz="0 0 0"/>
+		      <inertia ixx="1.0" ixy="0.0" ixz="0.0" iyy="1.0" iyz="0.0" izz="1.0"/>
+		    </inertial>
 		</link>
 		<!-- end of link list -->
@@ -155,4 +190,10 @@
 		</joint>
 		<!-- end of joint list -->
+	    <gazebo reference="${prefix}base_link">
+	      <material>blue</material>
+	    </gazebo>
+	    <gazebo reference="${prefix}link_s">
+	      <material>gray</material>
+	    </gazebo>
 	</xacro:macro>
 </robot>

File: vetex_support/urdf/vetex_macro.xacro (robot description, xacro)
@@ -17,4 +17,9 @@
         </geometry>
       </collision>
+      <inertial>
+        <mass value="0.1"/>
+        <origin xyz="0 0 0"/>
+        <inertia ixx="1.0" ixy="0.0" ixz="0.0" iyy="1.0" iyz="0.0" izz="1.0"/>
+      </inertial>
     </link>
     <link name="${prefix}base_footprint"/>
@@ -22,5 +27,6 @@
       <visual>
         <geometry>
-          <mesh filename="package://vetex_support/meshes/visual/left_front_wheel.stl" />
+          <cylinder length="0.2" radius="0.2"/>
+          <!-- <mesh filename="package://vetex_support/meshes/visual/left_front_wheel.stl" /> -->
         </geometry>
         <material name="euler_gray"/>
@@ -28,12 +34,19 @@
       <collision>
         <geometry>
-          <mesh filename="package://vetex_support/meshes/collision/left_front_wheel.stl" />
+          <cylinder length="0.2" radius="0.2"/>
+          <!-- <mesh filename="package://vetex_support/meshes/collision/left_front_wheel.stl" /> -->
         </geometry>
       </collision>
+      <inertial>
+        <mass value="0.1"/>
+        <origin xyz="0 0 0"/>
+        <inertia ixx="1.0" ixy="0.0" ixz="0.0" iyy="1.0" iyz="0.0" izz="1.0"/>
+      </inertial>
     </link>
     <link name="${prefix}left_rear_wheel">
       <visual>
         <geometry>
-          <mesh filename="package://vetex_support/meshes/visual/left_rear_wheel.stl" />
+          <cylinder length="0.2" radius="0.2"/>
+          <!-- <mesh filename="package://vetex_support/meshes/visual/left_rear_wheel.stl" /> -->
         </geometry>
         <material name="euler_gray"/>
@@ -41,7 +54,13 @@
       <collision>
         <geometry>
-          <mesh filename="package://vetex_support/meshes/collision/left_rear_wheel.stl" />
+          <cylinder length="0.2" radius="0.2"/>
+          <!-- <mesh filename="package://vetex_support/meshes/collision/left_rear_wheel.stl" /> -->
         </geometry>
       </collision>
+      <inertial>
+        <mass value="0.1"/>
+        <origin xyz="0 0 0"/>
+        <inertia ixx="1.0" ixy="0.0" ixz="0.0" iyy="1.0" iyz="0.0" izz="1.0"/>
+      </inertial>
     </link>
     <link name="${prefix}right_rear_wheel">
@@ -49,5 +68,6 @@
         <origin rpy="3.1415 0 0" />
         <geometry>
-          <mesh filename="package://vetex_support/meshes/visual/right_rear_wheel.stl" />
+          <cylinder length="0.2" radius="0.2"/>
+          <!-- <mesh filename="package://vetex_support/meshes/visual/right_rear_wheel.stl" /> -->
         </geometry>
         <material name="euler_gray"/>
@@ -56,7 +76,13 @@
         <origin rpy="3.1415 0 0" />
         <geometry>
-          <mesh filename="package://vetex_support/meshes/collision/right_rear_wheel.stl" />
+          <cylinder length="0.2" radius="0.2"/>
+          <!-- <mesh filename="package://vetex_support/meshes/collision/right_rear_wheel.stl" /> -->
         </geometry>
       </collision>
+      <inertial>
+        <mass value="0.1"/>
+        <origin xyz="0 0 0"/>
+        <inertia ixx="1.0" ixy="0.0" ixz="0.0" iyy="1.0" iyz="0.0" izz="1.0"/>
+      </inertial>
     </link>
     <link name="${prefix}right_front_wheel">
@@ -64,5 +90,6 @@
         <origin rpy="3.1415 0 0" />
         <geometry>
-          <mesh filename="package://vetex_support/meshes/visual/right_front_wheel.stl" />
+          <cylinder length="0.2" radius="0.2"/>
+          <!-- <mesh filename="package://vetex_support/meshes/visual/right_front_wheel.stl" /> -->
         </geometry>
         <material name="euler_gray"/>
@@ -71,7 +98,13 @@
         <origin rpy="3.1415 0 0" />
         <geometry>
-          <mesh filename="package://vetex_support/meshes/collision/right_front_wheel.stl" />
+          <cylinder length="0.2" radius="0.2"/>
+          <!-- <mesh filename="package://vetex_support/meshes/collision/right_front_wheel.stl" /> -->
         </geometry>
       </collision>
+      <inertial>
+        <mass value="0.1"/>
+        <origin xyz="0 0 0"/>
+        <inertia ixx="1.0" ixy="0.0" ixz="0.0" iyy="1.0" iyz="0.0" izz="1.0"/>
+      </inertial>
     </link>
     <!-- end of link list -->
@@ -83,5 +116,5 @@
     </joint>
     <joint name="${prefix}left_front_wheel_joint" type="continuous">
-      <origin xyz="0 0.58668 0.21577" rpy="0 1 0" />
+      <origin xyz="0 0.58668 0.21577" rpy="1.57 1 0" />
       <parent link="${prefix}base_link" />
       <child link="${prefix}left_front_wheel" />
@@ -90,5 +123,5 @@
     </joint>
     <joint name="${prefix}left_rear_wheel_joint" type="continuous">
-      <origin xyz="-2.0878 0.58642 0.21577" rpy="0 1 0" />
+      <origin xyz="-2.0878 0.58642 0.21577" rpy="1.57 1 0" />
       <parent link="${prefix}base_link" />
       <child link="${prefix}left_rear_wheel" />
@@ -97,5 +130,5 @@
     </joint>
     <joint name="${prefix}right_rear_wheel_joint" type="continuous">
-      <origin xyz="-2.0878 -0.58668 0.21577" rpy="0 1 0" />
+      <origin xyz="-2.0878 -0.58668 0.21577" rpy="1.57 1 0" />
       <parent link="${prefix}base_link" />
       <child link="${prefix}right_rear_wheel" />
@@ -104,5 +137,5 @@
     </joint>
     <joint name="${prefix}right_front_wheel_joint" type="continuous">
-      <origin xyz="0 -0.58642 0.21577" rpy="0 0 0" />
+      <origin xyz="0 -0.58642 0.21577" rpy="1.57 1 0" />
       <parent link="${prefix}base_link" />
       <child link="${prefix}right_front_wheel" />
