Commit message: Added friction plugin and gain values for the arm to move

File: euler_gazebo/urdf/euler.gazebo.component_macros.xacro (robot description, xacro)
@@ -31,4 +31,18 @@
        <actuator name="${prefix}${joint_name}_motor">
          <hardwareInterface>PositionJointInterface</hardwareInterface>
+         <mechanicalReduction>${reduction}</mechanicalReduction>
+       </actuator>
+       <motorTorqueConstant>${tc}</motorTorqueConstant>
+     </transmission>
+  </xacro:macro>
+  <!-- transmission EFFORT xacro -->
+  <xacro:macro name="gazebo_simple_effort_trans" params="prefix joint_name reduction tc">
+     <transmission name="${prefix}${joint_name}_trans">
+       <type>transmission_interface/SimpleTransmission</type>
+       <joint name="${prefix}${joint_name}">
+         <hardwareInterface>EffortJointInterface</hardwareInterface>
+       </joint>
+       <actuator name="${prefix}${joint_name}_motor">
+         <hardwareInterface>EffortJointInterface</hardwareInterface>
          <mechanicalReduction>${reduction}</mechanicalReduction>
        </actuator>
@@ -83,5 +97,5 @@
     <gazebo_joint prefix="${prefix}" joint_name="motoman_joint_b" kd="4" kp="10"/>
     <gazebo_joint prefix="${prefix}" joint_name="motoman_joint_t" kd="4" kp="10"/>
-    <gazebo_simple_pos_trans prefix="${prefix}" joint_name="motoman_joint_s" reduction="1" tc="1"/>
+<!--    <gazebo_simple_pos_trans prefix="${prefix}" joint_name="motoman_joint_s" reduction="1" tc="1"/>
     <gazebo_simple_pos_trans prefix="${prefix}" joint_name="motoman_joint_l" reduction="1" tc="1"/>
     <gazebo_simple_pos_trans prefix="${prefix}" joint_name="motoman_joint_u" reduction="1" tc="1"/>
@@ -89,4 +103,11 @@
     <gazebo_simple_pos_trans prefix="${prefix}" joint_name="motoman_joint_b" reduction="1" tc="1"/>
     <gazebo_simple_pos_trans prefix="${prefix}" joint_name="motoman_joint_t" reduction="1" tc="1"/>
+-->
+    <gazebo_simple_effort_trans prefix="${prefix}" joint_name="motoman_joint_s" reduction="1" tc="1"/>
+    <gazebo_simple_effort_trans prefix="${prefix}" joint_name="motoman_joint_l" reduction="1" tc="1"/>
+    <gazebo_simple_effort_trans prefix="${prefix}" joint_name="motoman_joint_u" reduction="1" tc="1"/>
+    <gazebo_simple_effort_trans prefix="${prefix}" joint_name="motoman_joint_r" reduction="1" tc="1"/>
+    <gazebo_simple_effort_trans prefix="${prefix}" joint_name="motoman_joint_b" reduction="1" tc="1"/>
+    <gazebo_simple_effort_trans prefix="${prefix}" joint_name="motoman_joint_t" reduction="1" tc="1"/>
   </xacro:macro>
   <!-- euler kinect xacro -->

File: euler_gazebo/urdf/euler_gazebo.xacro (robot description, xacro)
@@ -48,29 +48,25 @@
   <gazebo reference="vetex_right_rear_wheel">
     <material>Gazebo/Black</material>
-    <mu1 value="1.0" />
-    <mu2 value="1.0" />
-    <kp value="10000000.0" />
-    <kd value="1.0" />
+    <mu1 value="0.9" />
+    <mu2 value="0.9" />
+    <minDepth>0.0001</minDepth>
   </gazebo>
   <gazebo reference="vetex_right_front_wheel">
     <material>Gazebo/Black</material>
-    <mu1 value="1.0" />
-    <mu2 value="1.0" />
-    <kp value="10000000.0" />
-    <kd value="1.0" />
+    <mu1 value="0.9" />
+    <mu2 value="0.9" />
+    <minDepth>0.0001</minDepth>
   </gazebo>
   <gazebo reference="vetex_left_rear_wheel">
     <material>Gazebo/Black</material>
-    <mu1 value="1.0" />
-    <mu2 value="1.0" />
-    <kp value="10000000.0" />
-    <kd value="1.0" />
+    <mu1 value="0.9" />
+    <mu2 value="0.9" />
+    <minDepth>0.0001</minDepth>
   </gazebo>
   <gazebo reference="vetex_left_front_wheel">
     <material>Gazebo/Black</material>
-    <mu1 value="1.0" />
-    <mu2 value="1.0" />
-    <kp value="10000000.0" />
-    <kd value="1.0" />
+    <mu1 value="0.9" />
+    <mu2 value="0.9" />
+    <minDepth>0.0001</minDepth>
   </gazebo>
 </robot>

File: vetex_support/urdf/vetex_macro.xacro (robot description, xacro)
@@ -18,6 +18,6 @@
       </collision>
       <inertial>
-        <mass value="52.0"/>
-        <origin xyz="0 0 0"/>
+        <mass value="40.0"/>
+        <origin xyz="-1.04 0 0"/>
         <inertia ixx="1.0" ixy="0.0" ixz="0.0" iyy="1.0" iyz="0.0" izz="1.0"/>
       </inertial>
@@ -27,5 +27,4 @@
       <visual>
         <geometry>
-          <!--<cylinder length="0.2" radius="0.2"/>-->
           <mesh filename="package://vetex_support/meshes/visual/left_front_wheel.stl" />
         </geometry>
@@ -35,12 +34,10 @@
       </visual>
       <collision>
-        <origin xyz="0 -0.10 0" rpy="1.5708 0 0" />
         <geometry>
-          <cylinder length="0.2" radius="0.2"/>
-          <!--<mesh filename="package://vetex_support/meshes/collision/left_front_wheel.stl" /> -->
+          <mesh filename="package://vetex_support/meshes/collision/left_front_wheel.stl" />
         </geometry>
       </collision>
       <inertial>
-        <mass value="5.8517"/>
+        <mass value="4.0"/>
         <origin xyz="0 0 0"/>
         <inertia ixx="0.02467" ixy="0.0" ixz="0.0" iyy="0.04411" iyz="0.0" izz="0.02467"/>
@@ -50,5 +47,4 @@
       <visual>
         <geometry>
-          <!--<cylinder length="0.2" radius="0.2"/>-->
           <mesh filename="package://vetex_support/meshes/visual/left_rear_wheel.stl" />
         </geometry>
@@ -56,12 +52,10 @@
       </visual>
       <collision>
-        <origin xyz="0 -0.10 0" rpy="1.5708 0 0" />
         <geometry>
-          <cylinder length="0.2" radius="0.2"/>
-          <!-- <mesh filename="package://vetex_support/meshes/collision/left_rear_wheel.stl" /> -->
+          <mesh filename="package://vetex_support/meshes/collision/left_rear_wheel.stl" />
         </geometry>
       </collision>
       <inertial>
-        <mass value="5.8517"/>
+        <mass value="4.0"/>
         <origin xyz="0 0 0"/>
         <inertia ixx="0.02467" ixy="0.0" ixz="0.0" iyy="0.04411" iyz="0.0" izz="0.02467"/>
@@ -72,5 +66,4 @@
         <origin rpy="3.1415 0 0" />
         <geometry>
-          <!--<cylinder length="0.2" radius="0.2"/>-->
           <mesh filename="package://vetex_support/meshes/visual/right_rear_wheel.stl" />
         </geometry>
@@ -78,13 +71,11 @@
         </visual>
       <collision>
-        <origin xyz="0 0.10 0" rpy="1.5708 0 0" />
-        <!--<origin rpy="3.1415 0 0" />-->
+        <origin rpy="3.1415 0 0" />
         <geometry>
-          <cylinder length="0.2" radius="0.2"/>
-          <!-- <mesh filename="package://vetex_support/meshes/collision/right_rear_wheel.stl" /> -->
+          <mesh filename="package://vetex_support/meshes/collision/right_rear_wheel.stl" />
         </geometry>
       </collision>
       <inertial>
-        <mass value="5.8517"/>
+        <mass value="4.0"/>
         <origin xyz="0 0 0"/>
         <inertia ixx="0.02467" ixy="0.0" ixz="0.0" iyy="0.04411" iyz="0.0" izz="0.02467"/>
@@ -95,5 +86,4 @@
         <origin rpy="3.1415 0 0" />
         <geometry>
-          <!--<cylinder length="0.2" radius="0.2"/>-->
           <mesh filename="package://vetex_support/meshes/visual/right_front_wheel.stl" />
         </geometry>
@@ -101,13 +91,11 @@
       </visual>
       <collision>
-        <origin xyz="0 0.10 0" rpy="1.5708 0 0" />
-        <!--<origin rpy="3.1415 0 0" />-->
+        <origin rpy="3.1415 0 0" />
         <geometry>
-          <cylinder length="0.2" radius="0.2"/>
-          <!-- <mesh filename="package://vetex_support/meshes/collision/right_front_wheel.stl" /> -->
+          <mesh filename="package://vetex_support/meshes/collision/right_front_wheel.stl" />
         </geometry>
       </collision>
       <inertial>
-        <mass value="5.8517"/>
+        <mass value="4.0"/>
         <origin xyz="0 0 0"/>
         <inertia ixx="0.02467" ixy="0.0" ixz="0.0" iyy="0.04411" iyz="0.0" izz="0.02467"/>
@@ -117,5 +105,5 @@
     <!-- joint list -->
     <joint name="${prefix}to_footprint" type="fixed">
-      <origin xyz="-1.0439 0 0"/>
+      <origin xyz="0 0 0"/>
       <parent link="${prefix}base_link" />
       <child link="${prefix}base_footprint" />
@@ -127,5 +115,5 @@
       <child link="${prefix}left_front_wheel" />
       <axis xyz="0 1 0" />
-      <limit effort="20" velocity="3" />
+      <limit effort="50" velocity="3" />
     </joint>
     <joint name="${prefix}left_rear_wheel_joint" type="continuous">
@@ -135,5 +123,5 @@
       <child link="${prefix}left_rear_wheel" />
       <axis xyz="0 1 0" />
-      <limit effort="20" velocity="3" />
+      <limit effort="50" velocity="3" />
     </joint>
     <joint name="${prefix}right_rear_wheel_joint" type="continuous">
@@ -143,5 +131,5 @@
       <child link="${prefix}right_rear_wheel" />
       <axis xyz="0 1 0" />
-      <limit effort="20" velocity="3" />
+      <limit effort="50" velocity="3" />
     </joint>
     <joint name="${prefix}right_front_wheel_joint" type="continuous">
@@ -151,5 +139,5 @@
       <child link="${prefix}right_front_wheel" />
       <axis xyz="0 1 0" />
-      <limit effort="20" velocity="3" />
+      <limit effort="50" velocity="3" />
     </joint>
     <!-- end of joint list -->
