Commit message: Added color in Gazebo for Euler robot

File: euler_gazebo/urdf/euler_gazebo.xacro (robot description, xacro)
@@ -4,3 +4,54 @@
   <xacro:include filename="$(find euler_gazebo)/urdf/euler.gazebo.components.xacro"/>
   <xacro:include filename="$(find euler_gazebo)/urdf/euler.gazebo.controllers.xacro"/>
+  <gazebo reference="frame_left">
+    <material>Gazebo/Grey</material>
+  </gazebo>
+  <gazebo reference="frame_right">
+    <material>Gazebo/Grey</material>
+  </gazebo>
+  <gazebo reference="frame_top">
+    <material>Gazebo/Grey</material>
+  </gazebo>
+  <gazebo reference="vetex_base_link">
+    <material>Gazebo/Grey</material>
+  </gazebo>
+  <gazebo reference="motoman_base_link">
+    <material>Gazebo/Blue</material>
+  </gazebo>
+  <gazebo reference="motoman_link_s">
+    <material>Gazebo/Grey</material>
+  </gazebo>
+  <gazebo reference="motoman_link_l">
+    <material>Gazebo/Blue</material>
+  </gazebo>
+  <gazebo reference="motoman_link_r">
+    <material>Gazebo/Grey</material>
+  </gazebo>
+  <gazebo reference="motoman_link_b">
+    <material>Gazebo/Blue</material>
+  </gazebo>
+  <gazebo reference="eef_body">
+    <material>Gazebo/DarkGrey</material>
+  </gazebo>
+  <gazebo reference="sick_nav350">
+    <material>Gazebo/Blue</material>
+  </gazebo>
+  <gazebo reference="front_sick_s300">
+    <material>Gazebo/Yellow</material>
+  </gazebo>
+  <gazebo reference="rear_sick_s300">
+    <material>Gazebo/Yellow</material>
+  </gazebo>
+  <gazebo reference="vetex_right_rear_wheel">
+    <material>Gazebo/Black</material>
+  </gazebo>
+  <gazebo reference="vetex_right_front_wheel">
+    <material>Gazebo/Black</material>
+  </gazebo>
+  <gazebo reference="vetex_left_rear_wheel">
+    <material>Gazebo/Black</material>
+  </gazebo>
+  <gazebo reference="vetex_left_front_wheel">
+    <material>Gazebo/Black</material>
+  </gazebo>
 </robot>

Commit message: Add color black to Rviz wheels and set visuals to mecano wheels

File: euler_gazebo/urdf/euler_gazebo.xacro (robot description, xacro)
@@ -28,4 +28,7 @@
     <material>Gazebo/Grey</material>
   </gazebo>
+  <gazebo reference="motoman_link_u">
+    <material>Gazebo/Blue</material>
+  </gazebo>
   <gazebo reference="motoman_link_b">
     <material>Gazebo/Blue</material>

File: vetex_support/urdf/vetex_macro.xacro (robot description, xacro)
@@ -27,13 +27,15 @@
       <visual>
         <geometry>
-          <cylinder length="0.2" radius="0.2"/>
-          <!-- <mesh filename="package://vetex_support/meshes/visual/left_front_wheel.stl" /> -->
+          <!--<cylinder length="0.2" radius="0.2"/>-->
+          <mesh filename="package://vetex_support/meshes/visual/left_front_wheel.stl" />
         </geometry>
-        <material name="euler_gray"/>
+        <material name="euler_black">
+          <color rgba="0.01 0.01 0.01 1" />
+        </material>
       </visual>
       <collision>
         <geometry>
           <cylinder length="0.2" radius="0.2"/>
-          <!-- <mesh filename="package://vetex_support/meshes/collision/left_front_wheel.stl" /> -->
+          <!--<mesh filename="package://vetex_support/meshes/collision/left_front_wheel.stl" /> -->
         </geometry>
       </collision>
@@ -47,8 +49,8 @@
       <visual>
         <geometry>
-          <cylinder length="0.2" radius="0.2"/>
-          <!-- <mesh filename="package://vetex_support/meshes/visual/left_rear_wheel.stl" /> -->
+          <!--<cylinder length="0.2" radius="0.2"/>-->
+          <mesh filename="package://vetex_support/meshes/visual/left_rear_wheel.stl" />
         </geometry>
-        <material name="euler_gray"/>
+        <material name="euler_black"/>
       </visual>
       <collision>
@@ -68,8 +70,8 @@
         <origin rpy="3.1415 0 0" />
         <geometry>
-          <cylinder length="0.2" radius="0.2"/>
-          <!-- <mesh filename="package://vetex_support/meshes/visual/right_rear_wheel.stl" /> -->
+          <!--<cylinder length="0.2" radius="0.2"/>-->
+          <mesh filename="package://vetex_support/meshes/visual/right_rear_wheel.stl" />
         </geometry>
-        <material name="euler_gray"/>
+        <material name="euler_black"/>
         </visual>
       <collision>
@@ -90,8 +92,8 @@
         <origin rpy="3.1415 0 0" />
         <geometry>
-          <cylinder length="0.2" radius="0.2"/>
-          <!-- <mesh filename="package://vetex_support/meshes/visual/right_front_wheel.stl" /> -->
+          <!--<cylinder length="0.2" radius="0.2"/>-->
+          <mesh filename="package://vetex_support/meshes/visual/right_front_wheel.stl" />
         </geometry>
-        <material name="euler_gray"/>
+        <material name="euler_black"/>
       </visual>
       <collision>

Commit message: Added mu1 and mu2 to wheels. Turn but still not perfect

File: euler_gazebo/urdf/euler_gazebo.xacro (robot description, xacro)
@@ -48,13 +48,29 @@
   <gazebo reference="vetex_right_rear_wheel">
     <material>Gazebo/Black</material>
+    <mu1 value="1.0" />
+    <mu2 value="1.0" />
+    <kp value="10000000.0" />
+    <kd value="1.0" />
   </gazebo>
   <gazebo reference="vetex_right_front_wheel">
     <material>Gazebo/Black</material>
+    <mu1 value="1.0" />
+    <mu2 value="1.0" />
+    <kp value="10000000.0" />
+    <kd value="1.0" />
   </gazebo>
   <gazebo reference="vetex_left_rear_wheel">
     <material>Gazebo/Black</material>
+    <mu1 value="1.0" />
+    <mu2 value="1.0" />
+    <kp value="10000000.0" />
+    <kd value="1.0" />
   </gazebo>
   <gazebo reference="vetex_left_front_wheel">
     <material>Gazebo/Black</material>
+    <mu1 value="1.0" />
+    <mu2 value="1.0" />
+    <kp value="10000000.0" />
+    <kd value="1.0" />
   </gazebo>
 </robot>

File: vetex_support/urdf/vetex_macro.xacro (robot description, xacro)
@@ -35,5 +35,5 @@
       </visual>
       <collision>
-        <origin xyz="0 0 0" rpy="1.5708 0 0" />
+        <origin xyz="0 -0.10 0" rpy="1.5708 0 0" />
         <geometry>
           <cylinder length="0.2" radius="0.2"/>
@@ -44,5 +44,5 @@
         <mass value="5.8517"/>
         <origin xyz="0 0 0"/>
-        <inertia ixx="0.0501" ixy="0.0" ixz="0.0" iyy="0.0501" iyz="0.0" izz="0.0501"/>
+        <inertia ixx="0.02467" ixy="0.0" ixz="0.0" iyy="0.04411" iyz="0.0" izz="0.02467"/>
       </inertial>
     </link>
@@ -56,5 +56,5 @@
       </visual>
       <collision>
-        <origin xyz="0 0 0" rpy="1.5708 0 0" />
+        <origin xyz="0 -0.10 0" rpy="1.5708 0 0" />
         <geometry>
           <cylinder length="0.2" radius="0.2"/>
@@ -65,5 +65,5 @@
         <mass value="5.8517"/>
         <origin xyz="0 0 0"/>
-        <inertia ixx="0.0501" ixy="0.0" ixz="0.0" iyy="0.0501" iyz="0.0" izz="0.0501"/>
+        <inertia ixx="0.02467" ixy="0.0" ixz="0.0" iyy="0.04411" iyz="0.0" izz="0.02467"/>
       </inertial>
     </link>
@@ -78,5 +78,5 @@
         </visual>
       <collision>
-        <origin xyz="0 0 0" rpy="1.5708 0 0" />
+        <origin xyz="0 0.10 0" rpy="1.5708 0 0" />
         <!--<origin rpy="3.1415 0 0" />-->
         <geometry>
@@ -88,5 +88,5 @@
         <mass value="5.8517"/>
         <origin xyz="0 0 0"/>
-        <inertia ixx="0.0501" ixy="0.0" ixz="0.0" iyy="0.0501" iyz="0.0" izz="0.0501"/>
+        <inertia ixx="0.02467" ixy="0.0" ixz="0.0" iyy="0.04411" iyz="0.0" izz="0.02467"/>
       </inertial>
     </link>
@@ -101,5 +101,5 @@
       </visual>
       <collision>
-        <origin xyz="0 0 0" rpy="1.5708 0 0" />
+        <origin xyz="0 0.10 0" rpy="1.5708 0 0" />
         <!--<origin rpy="3.1415 0 0" />-->
         <geometry>
@@ -111,5 +111,5 @@
         <mass value="5.8517"/>
         <origin xyz="0 0 0"/>
-        <inertia ixx="0.0501" ixy="0.0" ixz="0.0" iyy="0.0501" iyz="0.0" izz="0.0501"/>
+        <inertia ixx="0.02467" ixy="0.0" ixz="0.0" iyy="0.04411" iyz="0.0" izz="0.02467"/>
       </inertial>
     </link>

Commit message: Added retrieval AT

File: euler_gazebo/urdf/euler_gazebo.xacro (robot description, xacro)
@@ -20,4 +20,7 @@
   <gazebo reference="vetex_base_link">
     <material>Gazebo/Grey</material>
+    <mu1 value="0.9" />
+    <mu2 value="0.9" />
+    <minDepth>0.0001</minDepth>
   </gazebo>
   <gazebo reference="motoman_base_link">

File: euler_support/urdf/euler_macro.xacro (robot description, xacro)
@@ -70,5 +70,5 @@
 			<origin xyz="0 0 0" rpy="0 0 0" />
 			<geometry>
-				<mesh filename="package://euler_support/meshes/collision/frame_top.stl" />
+				<mesh filename="package://euler_support/meshes/visual/frame_top.stl" /> <!-- The collision frame_top is oversized! Change -->
 			</geometry>
 		</collision>

Commit message: Added description for SICK sensors used in Euler

File: euler_gazebo/urdf/euler_gazebo.xacro (robot description, xacro)
@@ -5,7 +5,9 @@
   <xacro:include filename="$(find euler_gazebo)/urdf/euler.gazebo.controllers.xacro"/>
   <xacro:include filename="$(find euler_gazebo)/urdf/gazebo/sick_macros.gazebo.xacro" />
-  <!-- Sensors-->
-  <sick_s300_gazebo link="front_sick_s300" topic_name="front_sick_s300" />
+  <!-- Front sensor SICK S300 -->
+  <sick_s300_gazebo link="front_sick_s300" topic_name="front_sick_s300" visualize="true" />
+  <!-- Rear sensor SICK S300 -->
   <sick_s300_gazebo link="rear_sick_s300" topic_name="rear_sick_s300" />
+  <!-- Front, high-res sensor SICK Nav350 -->
   <sick_nav350_gazebo link="sick_nav350" topic_name="sick_nav350" />
   <gazebo reference="frame_left">

File: euler_gazebo/urdf/gazebo/sick_macros.gazebo.xacro (robot description, xacro)
@@ -1,9 +1,10 @@
 <?xml version="1.0"?>
 <robot xmlns:xacro="http://www.ros.org/wiki/xacro" name="sick_macros_gazebo" >
-  <xacro:macro name="sick_s300_gazebo" params="link topic_name">
+  <!-- Datasheet SICK S300: https://www.sick.com/media/pdf/6/46/846/dataSheet_S30B-3011GB_1057641_en.pdf -->
+  <xacro:macro name="sick_s300_gazebo" params="link topic_name visualize:=false">
     <gazebo reference="${link}">
       <sensor type="ray" name="${link}_sensor">
         <pose>0 0 0 0 0 0</pose>
-        <visualize>false</visualize>
+        <visualize>${visualize}</visualize>
         <update_rate>12.5</update_rate> <!-- Response time 80ms -->
         <ray>
@@ -31,10 +32,10 @@
     </gazebo>
   </xacro:macro>
-  <!-- Laser Scanner NAV350 Indoor Mid Range -->
-  <xacro:macro name="sick_nav350_gazebo" params="link topic_name">
+  <!-- Datasheet NAV350 Indoor Mid Range: https://sick-virginia.data.continum.net/media/pdf/1/41/041/dataSheet_NAV350-3232_1052928_en.pdf -->
+  <xacro:macro name="sick_nav350_gazebo" params="link topic_name visualize:=false">
     <gazebo reference="${link}">
       <sensor type="ray" name="${link}_sensor">
         <pose>0 0 0 0 0 0</pose>
-        <visualize>false</visualize>
+        <visualize>${visualize}</visualize>
         <update_rate>8.0</update_rate> <!-- 8Hz -->
         <ray>

Commit message: Fixed parameters for Asus Xtion to show up properly and align frames adequately

File: euler_gazebo/urdf/euler_gazebo.xacro (robot description, xacro)
@@ -5,10 +5,16 @@
   <xacro:include filename="$(find euler_gazebo)/urdf/euler.gazebo.controllers.xacro"/>
   <xacro:include filename="$(find euler_gazebo)/urdf/gazebo/sick_macros.gazebo.xacro" />
+  <xacro:include filename="$(find euler_gazebo)/urdf/gazebo/asus_xtion_macro.gazebo.xacro" />
   <!-- Front sensor SICK S300 -->
-  <sick_s300_gazebo link="front_sick_s300" topic_name="front_sick_s300" />
+  <!--<sick_s300_gazebo link="front_sick_s300" topic_name="front_sick_s300" />-->
   <!-- Rear sensor SICK S300 -->
-  <sick_s300_gazebo link="rear_sick_s300" topic_name="rear_sick_s300" />
+  <!--<sick_s300_gazebo link="rear_sick_s300" topic_name="rear_sick_s300" />-->
   <!-- Front, high-res sensor SICK Nav350 -->
-  <sick_nav350_gazebo link="sick_nav350" topic_name="sick_nav350" />
+  <!--<sick_nav350_gazebo link="sick_nav350" topic_name="sick_nav350" />-->
+  <!-- Asus Xtion -->
+  <asus_xtion_gazebo parent_link="asus_bodycenter" topic_name="asus" depth_frame="asus_depth_frame" />
+  <gazebo reference="asus_bodycenter">
+    <material>Gazebo/Black</material>
+  </gazebo>
   <gazebo reference="frame_left">
     <material>Gazebo/Grey</material>

File: euler_support/urdf/asus_xtion_pro.xacro (robot description, xacro)
@@ -6,10 +6,10 @@
   <link name="${sensor_name}_bodycenter">
     <visual>
-      <origin xyz="0 0 0 " rpy="0 0 0" />
+      <origin xyz="0 0 0 " rpy="-1.5708 0 -1.5708" />
       <geometry>
         <mesh filename="package://euler_support/meshes/visual/asus_sensor.stl"/>
       </geometry>
       <material name="lt_black">
-        <color rgba="0.3 0.3 0.3 1"/>
+        <color rgba="0.1 0.1 0.1 1"/>
       </material>
     </visual>
@@ -27,5 +27,5 @@
   </joint>
   <joint name="${sensor_name}_depth_joint" type="fixed">
-    <origin xyz="0.049 0 0" rpy="0 0 0" />
+    <origin xyz="0.049 0 0" rpy="-1.5708 0 -1.5708" />
     <parent link="${sensor_name}_bodycenter" />
     <child link="${sensor_name}_depth_frame" />
@@ -33,5 +33,5 @@
   <link name="${sensor_name}_depth_frame" />
   <joint name="${sensor_name}_rgb_joint" type="fixed">
-    <origin xyz="0.022 0 0" rpy="0 0 0" />
+    <origin xyz="0.022 0 0" rpy="-1.5708 0 -1.5708" />
     <parent link="${sensor_name}_bodycenter" />
     <child link="${sensor_name}_rgb_frame" />

File: euler_support/urdf/euler_macro.xacro (robot description, xacro)
@@ -8,5 +8,5 @@
 	<xacro:vetex prefix="vetex_" />
 	<xacro:motoman_mh5lf prefix="motoman_" />
-	<xacro:asus_xtion_pro sensor_name="" off_x="0.461" off_y="0" off_z="2.103" off_rr="1.5708" off_rp="1.8849" off_ry="0"/>
+	<xacro:asus_xtion_pro sensor_name="asus" off_x="0.461" off_y="0" off_z="2.103" off_rr="0" off_rp="0.31" off_ry="0"/> <!-- 1.5708 1.8849-->
 	<xacro:eef prefix=""/>
 	<!--link list -->
